File: Hardware/Electronics/CAD/SerialControllerBoard.kicad_sch (KiCad schematic)
At the start: 32 parts, among them J1 Conn_01x02, J10 Conn_01x04, J11 Conn_01x04, J2 Conn_01x03, J3 Conn_01x03, J4 Conn_01x03, J5 Conn_01x03, J6 Conn_01x02, J7 Conn_01x02, J8 Conn_02x03_Odd_Even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

Commit message: New controller board Layout with USB Hub and Arduino SoM
Parts:
- removed A1: Arduino_Nano_v3.x, Module:Arduino_Nano, symbol MCU_Module:Arduino_Nano_v3.x
- removed A2, A3: Pololu_Breakout_A4988, Module:Pololu_Breakout-16_15.2x20.3mm, symbol Driver_Motor:Pololu_Breakout_A4988
- removed J4: Conn_01x03, Connector_JST:JST_XH_B3B-XH-A_1x03_P2.50mm_Vertical, symbol Connector_Generic:Conn_01x03
- removed J8, J9: Conn_02x03_Odd_Even, Connector_PinHeader_2.54mm:PinHeader_2x03_P2.54mm_Vertical, symbol Connector_Generic:Conn_02x03_Odd_Even
- removed R10, R3, R4, R5, R6, R7, R8, R9: 10k, Resistor_SMD:R_0805_2012Metric_Pad1.20x1.40mm_HandSolder, symbol Device:R
- added A1: Arduino_Nano_v3.x, Module:Arduino_Nano_SoM, symbol Arduino_SoM:Arduino_Nano_v3.x
- added J7, J8, J9: Conn_01x04, Connector_JST:JST_PH_S4B-PH-SM4-TB_1x04-1MP_P2.00mm_Horizontal, symbol Connector_Generic:Conn_01x04
- added U1: FE11SX4, FE11SX4:FE11SX4, symbol FE11SX4:USB-HUB
- J1: footprint Connector_JST:JST_XH_B2B-XH-A_1x02_P2.50mm_Vertical -> JST-XH-Addon:JST_XH_S2B-XH-SM4-TB_1x02-1MP_P2.50mm_Horizontal
- J10, J11: footprint Connector_JST:JST_XH_B4B-XH-A_1x04_P2.50mm_Vertical -> Connector_JST:JST_PH_S4B-PH-SM4-TB_1x04-1MP_P2.00mm_Horizontal
- J2, J3: footprint Connector_JST:JST_XH_B3B-XH-A_1x03_P2.50mm_Vertical -> Connector_JST:JST_PH_S3B-PH-SM4-TB_1x03-1MP_P2.00mm_Horizontal
- J4: renamed from J5; footprint Connector_JST:JST_XH_B3B-XH-A_1x03_P2.50mm_Vertical -> Connector_JST:JST_PH_S3B-PH-SM4-TB_1x03-1MP_P2.00mm_Horizontal
- J5: renamed from J6; footprint Connector_JST:JST_XH_B2B-XH-A_1x02_P2.50mm_Vertical -> Connector_JST:JST_PH_S2B-PH-SM4-TB_1x02-1MP_P2.00mm_Horizontal
- J6: renamed from J7; footprint Connector_JST:JST_XH_B2B-XH-A_1x02_P2.50mm_Vertical -> Connector_JST:JST_PH_S2B-PH-SM4-TB_1x02-1MP_P2.00mm_Horizontal
Connections:
- net +5V: now also J11.1 (Pin_1), A1.27 (+5V), A1.31 (USB-V5), J7.1 (Pin_1), J8.1 (Pin_1), U1.1 (IN-5V), U1.13 (OUT3-5V), U1.5 (OUT1-5V), U1.9 (OUT2-5V)
- net GND: now also J10.2 (Pin_2), J11.4 (Pin_4), A1.29 (GND), A1.34 (USB-GND), A1.4 (GND), J7.4 (Pin_4), J8.4 (Pin_4), J9.2 (Pin_2), U1.12 (OUT2-GND), U1.16 (OUT3-GND), U1.4 (IN-GND), U1.8 (OUT1-GND)
- net VCC: now also J10.1 (Pin_1), J9.1 (Pin_1)
- net endstop-yaw: now also A1.19 (A0)
- net mag-sensor: now also A1.21 (A2)
- net trigger-primary: now also A1.6 (D3)
- net trigger-secondary: now also A1.7 (D4)
- net at J11.2 (Pin_2): now also U1.14 (OUT3-D-)
- net at J11.3 (Pin_3): now also U1.15 (OUT3-D+)
- net pitch-uart-tx: now reaches J10.4 (Pin_4)
- net pitch-uart-tx: now also A1.15 (D12)
- net pitch-uart-rx: now reaches J10.3 (Pin_3)
- net pitch-uart-rx: now also A1.14 (D11)
- net endstop-pitch-1 renamed endstop-pitch
- net endstop-pitch: now also A1.20 (A1)
- new net: J7.2 (Pin_2), U1.10 (OUT2-D-)
- new net: J7.3 (Pin_3), U1.11 (OUT2-D+)
- new net: J8.2 (Pin_2), U1.2 (IN-D-)
- new net: J8.3 (Pin_3), U1.3 (IN-D+)
- new net USB-D+: A1.33 (USB-D+), U1.7 (OUT1-D+)
- new net USB-D-: A1.32 (USB-D-), U1.6 (OUT1-D-)
- new net yaw-uart-rx: A1.9 (D6), J9.3 (Pin_3)
- new net yaw-uart-tx: A1.10 (D7), J9.4 (Pin_4)
- no-connect marks 0 -> 22
Other:
- note added: "Output FET Driver"
- note added: "Output Stepper Driver"
- note added: "USB-Hub"
- note removed: "Motor Driver"
- note removed: "Output Driver"
- moved on the sheet: J2, J3, J4
